File: hardware/OpenWeatherStation_MainBoard/connectors.kicad_sch (KiCad schematic)
At the start: 7 parts, among them J1 RJ45_LED_Shielded, J2 Conn_01x05_Pin, J4 Conn_02x07_Odd_Even

Commit message: poe wip
Parts:
- renumbered J1 to J3, R29 to R35, R28 to R36, R30 to R37
Connections:
- net GNDPWR is gone; now on net GND: J3.SH
Changed lines of the file:
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@@
     (stroke (width 0) (type default))
   )
-  (wire (pts (xy 74.93 105.41) (xy 74.93 104.14))
+  (wire (pts (xy 74.93 109.22) (xy 74.93 104.14))
     (stroke (width 0) (type default))
   )
@@
   )
   (wire (pts (xy 107.95 46.99) (xy 106.68 46.99))
-    (stroke (width 0) (type default))
-  )
-  (wire (pts (xy 74.93 105.41) (xy 69.85 105.41))
     (stroke (width 0) (type default))
   )
@@
   (symbol (lib_id "Device:R") (at 49.53 93.98 90) (mirror x) (unit 1)
     (in_bom yes) (on_board yes) (dnp no) (fields_autoplaced)
-    (property "Reference" "R28" (at 50.8 91.44 0)
+    (property "Reference" "R36" (at 50.8 91.44 0)
       (effects (font (size 1.27 1.27)) (justify right))
     )
@@
     (instances
       (project "OpenWeatherStation_MainBoard"
-        (path "/698c4dde-56a2-4dd1-89d2-180a09a5dfe9/7c03bbc1-3816-4af6-9da6-b1bc735a9c60"
-          (reference "R28") (unit 1)
-        )
         (path "/698c4dde-56a2-4dd1-89d2-180a09a5dfe9/353c80a6-1831-46d1-b79a-6f2062aa4dd2"
           (reference "R36") (unit 1)
@@
     )
   )
+  (symbol (lib_id "power:GND") (at 74.93 109.22 0) (unit 1)
+    (in_bom yes) (on_board yes) (dnp no) (fields_autoplaced)
+    (property "Reference" "#PWR036" (at 74.93 115.57 0)
+      (effects (font (size 1.27 1.27)) hide)
+    )
+    (property "Value" "GND" (at 74.93 114.3 0)
+      (effects (font (size 1.27 1.27)))
+    )
+    (property "Footprint" "" (at 74.93 109.22 0)
+      (effects (font (size 1.27 1.27)) hide)
+    )
+    (property "Datasheet" "" (at 74.93 109.22 0)
+      (effects (font (size 1.27 1.27)) hide)
+    )
+    (pin "1")
+    (instances
+      (project "OpenWeatherStation_MainBoard"
+        (path "/698c4dde-56a2-4dd1-89d2-180a09a5dfe9/353c80a6-1831-46d1-b79a-6f2062aa4dd2"
+          (reference "#PWR036") (unit 1)
+        )
+      )
+    )
+  )
   (symbol (lib_id "Device:R") (at 49.53 78.74 90) (mirror x) (unit 1)
     (in_bom yes) (on_board yes) (dnp no) (fields_autoplaced)
-    (property "Reference" "R29" (at 50.8 76.2 0)
+    (property "Reference" "R35" (at 50.8 76.2 0)
       (effects (font (size 1.27 1.27)) (justify right))
     )
@@
     (instances
       (project "OpenWeatherStation_MainBoard"
-        (path "/698c4dde-56a2-4dd1-89d2-180a09a5dfe9/7c03bbc1-3816-4af6-9da6-b1bc735a9c60"
-          (reference "R29") (unit 1)
-        )
         (path "/698c4dde-56a2-4dd1-89d2-180a09a5dfe9/353c80a6-1831-46d1-b79a-6f2062aa4dd2"
           (reference "R35") (unit 1)
@@
   (symbol (lib_id "power:GND") (at 45.72 78.74 270) (mirror x) (unit 1)
     (in_bom yes) (on_board yes) (dnp no) (fields_autoplaced)
-    (property "Reference" "#PWR024" (at 39.37 78.74 0)
+    (property "Reference" "#PWR033" (at 39.37 78.74 0)
       (effects (font (size 1.27 1.27)) hide)
     )
@@
     (instances
       (project "OpenWeatherStation_MainBoard"
-        (path "/698c4dde-56a2-4dd1-89d2-180a09a5dfe9/7c03bbc1-3816-4af6-9da6-b1bc735a9c60"
-          (reference "#PWR024") (unit 1)
-        )
         (path "/698c4dde-56a2-4dd1-89d2-180a09a5dfe9/353c80a6-1831-46d1-b79a-6f2062aa4dd2"
           (reference "#PWR033") (unit 1)
@@
   (symbol (lib_id "power:GND") (at 54.61 109.22 0) (mirror y) (unit 1)
     (in_bom yes) (on_board yes) (dnp no) (fields_autoplaced)
-    (property "Reference" "#PWR025" (at 54.61 115.57 0)
+    (property "Reference" "#PWR035" (at 54.61 115.57 0)
       (effects (font (size 1.27 1.27)) hide)
     )
@@
     (instances
       (project "OpenWeatherStation_MainBoard"
-        (path "/698c4dde-56a2-4dd1-89d2-180a09a5dfe9/7c03bbc1-3816-4af6-9da6-b1bc735a9c60"
-          (reference "#PWR025") (unit 1)
-        )
         (path "/698c4dde-56a2-4dd1-89d2-180a09a5dfe9/353c80a6-1831-46d1-b79a-6f2062aa4dd2"
           (reference "#PWR035") (unit 1)
@@
   (symbol (lib_id "Device:R") (at 54.61 105.41 0) (unit 1)
     (in_bom yes) (on_board yes) (dnp no) (fields_autoplaced)
-    (property "Reference" "R30" (at 57.15 104.14 0)
+    (property "Reference" "R37" (at 57.15 104.14 0)
       (effects (font (size 1.27 1.27)) (justify left))
     )
@@
     (instances
       (project "OpenWeatherStation_MainBoard"
-        (path "/698c4dde-56a2-4dd1-89d2-180a09a5dfe9/7c03bbc1-3816-4af6-9da6-b1bc735a9c60"
-          (reference "R30") (unit 1)
-        )
         (path "/698c4dde-56a2-4dd1-89d2-180a09a5dfe9/353c80a6-1831-46d1-b79a-6f2062aa4dd2"
           (reference "R37") (unit 1)
-        )
-      )
-    )
-  )
-  (symbol (lib_id "power:GNDPWR") (at 69.85 105.41 0) (unit 1)
-    (in_bom yes) (on_board yes) (dnp no) (fields_autoplaced)
-    (property "Reference" "#PWR01" (at 69.85 110.49 0)
-      (effects (font (size 1.27 1.27)) hide)
-    )
-    (property "Value" "GNDPWR" (at 69.723 108.9486 0)
-      (effects (font (size 1.27 1.27)))
-    )
-    (property "Footprint" "" (at 69.85 106.68 0)
-      (effects (font (size 1.27 1.27)) hide)
-    )
-    (property "Datasheet" "" (at 69.85 106.68 0)
-      (effects (font (size 1.27 1.27)) hide)
-    )
-    (pin "1")
-    (instances
-      (project "OpenWeatherStation_MainBoard"
-        (path "/698c4dde-56a2-4dd1-89d2-180a09a5dfe9/7c03bbc1-3816-4af6-9da6-b1bc735a9c60"
-          (reference "#PWR01") (unit 1)
-        )
-        (path "/698c4dde-56a2-4dd1-89d2-180a09a5dfe9/353c80a6-1831-46d1-b79a-6f2062aa4dd2"
-          (reference "#PWR036") (unit 1)
         )
       )
@@
   (symbol (lib_id "Connector:RJ45_LED_Shielded") (at 74.93 91.44 0) (unit 1)
     (in_bom yes) (on_board yes) (dnp no) (fields_autoplaced)
-    (property "Reference" "J1" (at 74.93 75.16 0)
+    (property "Reference" "J3" (at 74.93 75.16 0)
       (effects (font (size 1.27 1.27)))
     )
@@
     (instances
       (project "OpenWeatherStation_MainBoard"
-        (path "/698c4dde-56a2-4dd1-89d2-180a09a5dfe9/7c03bbc1-3816-4af6-9da6-b1bc735a9c60"
-          (reference "J1") (unit 1)
-        )
         (path "/698c4dde-56a2-4dd1-89d2-180a09a5dfe9/353c80a6-1831-46d1-b79a-6f2062aa4dd2"
           (reference "J3") (unit 1)
@@
   (symbol (lib_id "power:GND") (at 45.72 93.98 270) (mirror x) (unit 1)
     (in_bom yes) (on_board yes) (dnp no) (fields_autoplaced)
-    (property "Reference" "#PWR023" (at 39.37 93.98 0)
+    (property "Reference" "#PWR034" (at 39.37 93.98 0)
       (effects (font (size 1.27 1.27)) hide)
     )
@@
     (instances
       (project "OpenWeatherStation_MainBoard"
-        (path "/698c4dde-56a2-4dd1-89d2-180a09a5dfe9/7c03bbc1-3816-4af6-9da6-b1bc735a9c60"
-          (reference "#PWR023") (unit 1)
-        )
         (path "/698c4dde-56a2-4dd1-89d2-180a09a5dfe9/353c80a6-1831-46d1-b79a-6f2062aa4dd2"
           (reference "#PWR034") (unit 1)

Commit message: electrical design wip
Parts:
- J4: footprint (none) -> Connector_PinHeader_1.27mm:PinHeader_2x07_P1.27mm_Vertical
- R28: value 100 -> 100R; footprint (none) -> Resistor_SMD:R_0603_1608Metric
- R35, R36: value 270 -> 270R; footprint (none) -> Resistor_SMD:R_0603_1608Metric
- R37: footprint (none) -> Resistor_SMD:R_0603_1608Metric
Other:
- company: (none) -> Vital Septfonds
- title: (none) -> Open Wheather Station
Changed lines of the file:
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@@
 (kicad_sch (version 20230121) (generator eeschema)
   (paper "A4")
+  (title_block
+    (title "Open Wheather Station")
+    (date "2024-01-02")
+    (rev "1.0")
+    (company "Vital Septfonds")
+  )
   (junction (at 121.92 41.91) (diameter 0) (color 0 0 0 0)
   )
@@
       (effects (font (size 1.27 1.27)) (justify right))
     )
-    (property "Value" "270" (at 48.26 91.44 0)
+    (property "Value" "270R" (at 48.26 91.44 0)
       (effects (font (size 1.27 1.27)) (justify right))
     )
-    (property "Footprint" "" (at 49.53 92.202 90)
+    (property "Footprint" "Resistor_SMD:R_0603_1608Metric" (at 49.53 92.202 90)
       (effects (font (size 1.27 1.27)) hide)
     )
@@
       (effects (font (size 1.27 1.27)) (justify right))
     )
-    (property "Value" "270" (at 48.26 76.2 0)
+    (property "Value" "270R" (at 48.26 76.2 0)
       (effects (font (size 1.27 1.27)) (justify right))
     )
-    (property "Footprint" "" (at 49.53 76.962 90)
+    (property "Footprint" "Resistor_SMD:R_0603_1608Metric" (at 49.53 76.962 90)
       (effects (font (size 1.27 1.27)) hide)
     )
@@
       (effects (font (size 1.27 1.27)))
     )
-    (property "Footprint" "" (at 128.27 41.91 0)
+    (property "Footprint" "Connector_PinHeader_1.27mm:PinHeader_2x07_P1.27mm_Vertical" (at 128.27 41.91 0)
       (effects (font (size 1.27 1.27)) hide)
     )
@@
       (effects (font (size 1.27 1.27)) (justify left))
     )
-    (property "Footprint" "" (at 52.832 105.41 90)
+    (property "Footprint" "Resistor_SMD:R_0603_1608Metric" (at 52.832 105.41 90)
       (effects (font (size 1.27 1.27)) hide)
     )
@@
       (effects (font (size 1.27 1.27)))
     )
-    (property "Value" "100" (at 111.76 52.07 90)
-      (effects (font (size 1.27 1.27)))
-    )
-    (property "Footprint" "" (at 111.76 48.768 90)
-      (effects (font (size 1.27 1.27)) hide)
-    )
+    (property "Value" "100R" (at 111.76 52.07 90)
+      (effects (font (size 1.27 1.27)))
+    )
+    (property "Footprint" "Resistor_SMD:R_0603_1608Metric" (at 111.76 48.768 90)
+      (effects (font (size 1.27 1.27)) hide)
+    )

Commit message: update elec
Other:
- moved on the sheet: J4, R28

Commit message: udpate pcb design
Parts:
- J2: footprint (none) -> Connector_JST:JST_XH_B5B-XH-A_1x05_P2.50mm_Vertical
- J3: footprint (none) -> Connector_RJ:RJ45_Amphenol_RJHSE538X
Changed lines of the file:
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@@
       (effects (font (size 1.27 1.27)))
     )
-    (property "Footprint" "" (at 46.99 43.18 0)
+    (property "Footprint" "Connector_JST:JST_XH_B5B-XH-A_1x05_P2.50mm_Vertical" (at 46.99 43.18 0)
       (effects (font (size 1.27 1.27)) hide)
     )
@@
       (effects (font (size 1.27 1.27)))
     )
-    (property "Footprint" "" (at 74.93 90.805 90)
-      (effects (font (size 1.27 1.27)) hide)
-    )
+    (property "Footprint" "Connector_RJ:RJ45_Amphenol_RJHSE538X" (at 74.93 90.805 90)
+      (effects (font (size 1.27 1.27)) hide)
+    )
