File: hardware/OpenWeatherStation_MainBoard/ethernet.kicad_sch (KiCad schematic)
At the start: 0 parts

Commit message: update board schematics (sensors, ethernet ...)
Parts:
- added C23, C24: 30p, symbol Device:C
- added C25, C28, C29, C30, C31, C32: 100n, symbol Device:C
- added C26: 1u, symbol Device:C
- added C27: 470p, symbol Device:C
- added C33: 10u, symbol Device:C_Polarized
- added FB1: FerriteBead, symbol Device:FerriteBead
- added R18, R19, R2, R24: 33, symbol Device:R
- added R20, R21, R22, R25, R26: 10k, symbol Device:R
- added R23: 1k5, symbol Device:R
- added R27: 12k1, symbol Device:R
- added R31, R32, R33, R34: 50, symbol Device:R
- added U7: USBLC6-4SC6, Package_TO_SOT_SMD:SOT-23-6, symbol Power_Protection:USBLC6-4SC6
- added U8: LAN8742A, Package_DFN_QFN:VQFN-24-1EP_4x4mm_P0.5mm_EP2.5x2.5mm_ThermalVias, symbol Interface_Ethernet:LAN8742A
- added Y1: Crystal, symbol Device:Crystal
Connections:
- new net: R18.2, R21.1, U8.7 (RXD1/MODE1)
- new net: R19.2, R22.1, U8.11 (CRS_DV/MODE2)
- new net: R24.2, R25.1, U8.14 (~{INT}/REFCLKO)
- new net: R27.1, U8.24 (RBIAS)
- new net: R2.2, R20.1, U8.8 (RXD0/MODE0)
- new net: R26.1, U8.10 (RXER/PHYAD0)
- new net: C24.1, U8.4 (XTAL2), Y1.1
- new net: C23.1, U8.5 (XTAL1/CLKIN), Y1.2
- new net: C26.1, C27.2, U8.6 (VDDCR)
- new net +3V3: C28.1, FB1.2, R20.2, R21.2, R22.2, R23.2, R25.2, U8.9 (VDDIO)
- new net CRC_DV: R19.1
- new net CT: C25.1, C29.1, C30.1, C31.1, C32.1, C33.1, FB1.1, R31.1, R32.1, R33.1, R34.1, U7.5 (VBUS), U8.1 (VDD2A), U8.19 (VDD1A)
- new net GND: C23.2, C24.2, C25.2, C26.2, C27.1, C28.2, C29.2, C30.2, C31.2, C32.2, C33.2, R26.2, R27.2, U7.2 (GND), U8.25 (VSS)
- new net LED_GREEN: U8.2 (LED2/~{INTSEL})
- new net LED_YELLOW: U8.3 (LED1/REGOFF)
- new net MDC: U8.13 (MDC)
- new net MDIO: R23.1, U8.12 (MDIO)
- new net RD+: R32.2, U7.1 (I/O1), U8.23 (RXP)
- new net RD-: R31.2, U7.6 (I/O4), U8.22 (RXN)
- new net REF_CLK: R24.1
- new net RXD0: R2.1
- new net RXD1: R18.1
- new net TD+: R34.2, U7.3 (I/O2), U8.21 (TXP)
- new net TD-: R33.2, U7.4 (I/O3), U8.20 (TXN)
- new net TXD0: U8.17 (TXD0)
- new net TXD1: U8.18 (TXD1)
- new net TX_EN: U8.16 (TXEN)
Other:
- note added: "Diff pair"

Commit message: fix hierarchical bus
Connections:
- net CRC_DV renamed ETH.CRC_DV
- net CT renamed ETH_DATA.CT
- net LED_GREEN renamed ETH_STATUS.LED_GREEN
- net LED_YELLOW renamed ETH_STATUS.LED_YELLOW
- net MDC renamed ETH.MDC
- net MDIO renamed ETH.MDIO
- net RD+ renamed ETH_DATA.RD+
- net RD- renamed ETH_DATA.RD-
- net REF_CLK renamed ETH.REF_CLK
- net RXD0 renamed ETH.RXD0
- net RXD1 renamed ETH.RXD1
- net TD+ renamed ETH_DATA.TD+
- net TD- renamed ETH_DATA.TD-
- net TXD0 renamed ETH.TXD0
- net TXD1 renamed ETH.TXD1
- net TX_EN renamed ETH.TX_EN
Other:
- moved on the sheet: C28

Commit message: schematic update
Connections:
- net NRST: now reaches U8.15 (~{RST})
Changed lines of the file:
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@@
+    (stroke (width 0) (type default))
+  )
+  (wire (pts (xy 120.65 99.06) (xy 128.27 99.06))
     (stroke (width 0) (type default))
   )
@@
     (effects (font (size 1.27 1.27)) (justify right))
   )
+  (hierarchical_label "NRST" (shape input) (at 120.65 99.06 180) (fields_autoplaced)
+    (effects (font (size 1.27 1.27)) (justify right))
+  )

Commit message: electrical design wip
Parts:
- C23, C24: value 30p -> 30pF; footprint (none) -> Capacitor_SMD:C_0603_1608Metric
- C25, C28, C29, C30, C31, C32: value 100n -> 100nF; footprint (none) -> Capacitor_SMD:C_0603_1608Metric
- C26: value 1u -> 1uF; footprint (none) -> Capacitor_SMD:C_0603_1608Metric
- C27: value 470p -> 470pF; footprint (none) -> Capacitor_SMD:C_0603_1608Metric
- C33: value 10u -> 10uF; footprint (none) -> Capacitor_SMD:C_0603_1608Metric
- R18, R19, R2, R24: value 33 -> 33R; footprint (none) -> Resistor_SMD:R_0603_1608Metric
- R20, R21, R22, R23, R25, R26, R27: footprint (none) -> Resistor_SMD:R_0603_1608Metric
- R31, R32, R33, R34: value 50 -> 50R; footprint (none) -> Resistor_SMD:R_0603_1608Metric
- Y1: footprint (none) -> Crystal:Crystal_SMD_Abracon_ABM3B-4Pin_5.0x3.2mm
Other:
- company: (none) -> Vital Septfonds
- title: (none) -> Open Wheather Station

Commit message: update elec
Changed lines of the file:
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@@
   (junction (at 101.6 39.37) (diameter 0) (color 0 0 0 0)
   )
+  (junction (at 143.51 58.42) (diameter 0) (color 0 0 0 0)
+  )
   (junction (at 203.2 76.2) (diameter 0) (color 0 0 0 0)
   )
@@
   (junction (at 237.49 39.37) (diameter 0) (color 0 0 0 0)
   )
+  (junction (at 146.05 39.37) (diameter 0) (color 0 0 0 0)
+  )
   (junction (at 269.24 39.37) (diameter 0) (color 0 0 0 0)
   )
@@
   (junction (at 256.54 39.37) (diameter 0) (color 0 0 0 0)
   )
+  (junction (at 157.48 39.37) (diameter 0) (color 0 0 0 0)
+  )
   (junction (at 186.69 78.74) (diameter 0) (color 0 0 0 0)
   )
@@
   (junction (at 252.73 39.37) (diameter 0) (color 0 0 0 0)
   )
+  (junction (at 148.59 127) (diameter 0) (color 0 0 0 0)
+  )
   (junction (at 254 54.61) (diameter 0) (color 0 0 0 0)
   )
@@
     (stroke (width 0) (type default))
   )
-  (wire (pts (xy 151.13 39.37) (xy 173.99 39.37))
+  (wire (pts (xy 151.13 39.37) (xy 157.48 39.37))
     (stroke (width 0) (type default))
   )
@@
     (stroke (width 0) (type default))
   )
+  (wire (pts (xy 157.48 39.37) (xy 173.99 39.37))
+    (stroke (width 0) (type default))
+  )
   (wire (pts (xy 116.84 66.04) (xy 116.84 88.9))
     (stroke (width 0) (type default))
@@
     (stroke (width 0) (type default))
   )
-  (wire (pts (xy 148.59 116.84) (xy 148.59 134.62))
+  (wire (pts (xy 148.59 116.84) (xy 148.59 127))
     (stroke (width 0) (type default))
   )
@@
   )
   (wire (pts (xy 27.94 76.2) (xy 128.27 76.2))
+    (stroke (width 0) (type default))
+  )
+  (wire (pts (xy 148.59 127) (xy 148.59 134.62))
     (stroke (width 0) (type default))
   )
@@
     )
   )
+  (symbol (lib_id "power:PWR_FLAG") (at 143.51 58.42 90) (unit 1)
+    (in_bom yes) (on_board yes) (dnp no) (fields_autoplaced)
+    (property "Reference" "#FLG04" (at 141.605 58.42 0)
+      (effects (font (size 1.27 1.27)) hide)
+    )
+    (property "Value" "PWR_FLAG" (at 139.7 58.42 90)
+      (effects (font (size 1.27 1.27)) (justify left))
+    )
+    (property "Footprint" "" (at 143.51 58.42 0)
+      (effects (font (size 1.27 1.27)) hide)
+    )
+    (property "Datasheet" "~" (at 143.51 58.42 0)
+      (effects (font (size 1.27 1.27)) hide)
+    )
+    (pin "1")
+    (instances
+      (project "OpenWeatherStation_MainBoard"
+        (path "/698c4dde-56a2-4dd1-89d2-180a09a5dfe9/31524387-a762-4425-ba1e-acf8940bc01b"
+          (reference "#FLG04") (unit 1)
+        )
+      )
+    )
+  )
   (symbol (lib_id "Device:R") (at 87.63 86.36 270) (unit 1)
     (in_bom yes) (on_board yes) (dnp no) (fields_autoplaced)
@@
         (path "/698c4dde-56a2-4dd1-89d2-180a09a5dfe9/31524387-a762-4425-ba1e-acf8940bc01b"
           (reference "#PWR030") (unit 1)
+        )
+      )
+    )
+  )
+  (symbol (lib_id "power:PWR_FLAG") (at 157.48 39.37 0) (unit 1)
+    (in_bom yes) (on_board yes) (dnp no) (fields_autoplaced)
+    (property "Reference" "#FLG05" (at 157.48 37.465 0)
+      (effects (font (size 1.27 1.27)) hide)
+    )
+    (property "Value" "PWR_FLAG" (at 157.48 34.29 0)
+      (effects (font (size 1.27 1.27)))
+    )
+    (property "Footprint" "" (at 157.48 39.37 0)
+      (effects (font (size 1.27 1.27)) hide)
+    )
+    (property "Datasheet" "~" (at 157.48 39.37 0)
+      (effects (font (size 1.27 1.27)) hide)
+    )
+    (pin "1")
+    (instances
+      (project "OpenWeatherStation_MainBoard"
+        (path "/698c4dde-56a2-4dd1-89d2-180a09a5dfe9/31524387-a762-4425-ba1e-acf8940bc01b"
+          (reference "#FLG05") (unit 1)
         )
       )
@@
     )
   )
+  (symbol (lib_id "power:PWR_FLAG") (at 146.05 39.37 0) (unit 1)
+    (in_bom yes) (on_board yes) (dnp no) (fields_autoplaced)
+    (property "Reference" "#FLG06" (at 146.05 37.465 0)
+      (effects (font (size 1.27 1.27)) hide)
+    )
+    (property "Value" "PWR_FLAG" (at 146.05 34.29 0)
+      (effects (font (size 1.27 1.27)))
+    )
+    (property "Footprint" "" (at 146.05 39.37 0)
+      (effects (font (size 1.27 1.27)) hide)
+    )
+    (property "Datasheet" "~" (at 146.05 39.37 0)
+      (effects (font (size 1.27 1.27)) hide)
+    )
+    (pin "1")
+    (instances
+      (project "OpenWeatherStation_MainBoard"
+        (path "/698c4dde-56a2-4dd1-89d2-180a09a5dfe9/31524387-a762-4425-ba1e-acf8940bc01b"
+          (reference "#FLG06") (unit 1)
+        )
+      )
+    )
+  )
   (symbol (lib_id "Device:R") (at 62.23 81.28 90) (unit 1)
     (in_bom yes) (on_board yes) (dnp no) (fields_autoplaced)
@@
         )
       )
+    )
+  )
+  (symbol (lib_id "power:PWR_FLAG") (at 148.59 127 270) (unit 1)
+    (in_bom yes) (on_board yes) (dnp no) (fields_autoplaced)
+    (property "Reference" "#FLG03" (at 150.495 127 0)
+      (effects (font (size 1.27 1.27)) hide)
+    )
+    (property "Value" "PWR_FLAG" (at 152.4 127 90)
+      (effects (font (size 1.27 1.27)) (justify left))
+    )
+    (property "Footprint" "" (at 148.59 127 0)
+      (effects (font (size 1.27 1.27)) hide)
+    )
+    (property "Datasheet" "~" (at 148.59 127 0)
+      (effects (font (size 1.27 1.27)) hide)
+    )
+    (pin "1")
+    (instances
+      (project "OpenWeatherStation_MainBoard"
+        (path "/698c4dde-56a2-4dd1-89d2-180a09a5dfe9/31524387-a762-4425-ba1e-acf8940bc01b"
+          (reference "#FLG03") (unit 1)
+        )
+      )

Commit message: udpate pcb design
Parts:
- FB1: footprint (none) -> Capacitor_SMD:C_0603_1608Metric
Changed lines of the file:
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@@
       (effects (font (size 1.27 1.27)))
     )
-    (property "Footprint" "" (at 250.952 31.75 90)
+    (property "Footprint" "Capacitor_SMD:C_0603_1608Metric" (at 250.952 31.75 90)
       (effects (font (size 1.27 1.27)) hide)
     )
