File: hardware/OpenWeatherStation_MainBoard/sensors.kicad_sch (KiCad schematic)
At the start: 5 parts, among them U2 FXPS7115D4, U3 HTU21D

Commit message: update elec
Other:
- moved on the sheet: C21, U3
Changed lines of the file:
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@@
     (company "Vital Septfonds")
   )
-  (junction (at 71.12 72.39) (diameter 0) (color 0 0 0 0)
+  (junction (at 71.12 69.85) (diameter 0) (color 0 0 0 0)
   )
   (junction (at 63.5 97.79) (diameter 0) (color 0 0 0 0)
@@
   (junction (at 60.96 146.05) (diameter 0) (color 0 0 0 0)
   )
-  (junction (at 71.12 54.61) (diameter 0) (color 0 0 0 0)
+  (junction (at 71.12 52.07) (diameter 0) (color 0 0 0 0)
   )
   (junction (at 63.5 146.05) (diameter 0) (color 0 0 0 0)
@@
     (stroke (width 0) (type default))
   )
+  (bus_entry (at 106.68 60.96) (size 2.54 2.54)
+    (stroke (width 0) (type default))
+  )
+  (bus_entry (at 106.68 125.73) (size 2.54 2.54)
+    (stroke (width 0) (type default))
+  )
   (bus_entry (at 106.68 63.5) (size 2.54 2.54)
     (stroke (width 0) (type default))
   )
-  (bus_entry (at 106.68 125.73) (size 2.54 2.54)
-    (stroke (width 0) (type default))
-  )
-  (bus_entry (at 106.68 66.04) (size 2.54 2.54)
-    (stroke (width 0) (type default))
-  )
   (wire (pts (xy 60.96 146.05) (xy 60.96 147.32))
     (stroke (width 0) (type default))
@@
     (stroke (width 0) (type default))
   )
-  (bus (pts (xy 109.22 66.04) (xy 109.22 68.58))
+  (bus (pts (xy 109.22 63.5) (xy 109.22 66.04))
     (stroke (width 0) (type default))
   )
@@
     (stroke (width 0) (type default))
   )
-  (wire (pts (xy 71.12 72.39) (xy 71.12 74.93))
+  (wire (pts (xy 71.12 69.85) (xy 71.12 72.39))
     (stroke (width 0) (type default))
   )
@@
     (stroke (width 0) (type default))
   )
-  (wire (pts (xy 71.12 52.07) (xy 71.12 54.61))
-    (stroke (width 0) (type default))
-  )
-  (wire (pts (xy 59.69 67.31) (xy 59.69 72.39))
+  (wire (pts (xy 71.12 49.53) (xy 71.12 52.07))
+    (stroke (width 0) (type default))
+  )
+  (wire (pts (xy 59.69 64.77) (xy 59.69 69.85))
     (stroke (width 0) (type default))
   )
@@
     (stroke (width 0) (type default))
   )
-  (wire (pts (xy 59.69 72.39) (xy 71.12 72.39))
-    (stroke (width 0) (type default))
-  )
-  (wire (pts (xy 59.69 54.61) (xy 71.12 54.61))
-    (stroke (width 0) (type default))
-  )
-  (bus (pts (xy 109.22 68.58) (xy 109.22 123.19))
+  (wire (pts (xy 59.69 69.85) (xy 71.12 69.85))
+    (stroke (width 0) (type default))
+  )
+  (wire (pts (xy 59.69 52.07) (xy 71.12 52.07))
+    (stroke (width 0) (type default))
+  )
+  (bus (pts (xy 109.22 66.04) (xy 109.22 123.19))
     (stroke (width 0) (type default))
   )
@@
     (stroke (width 0) (type default))
   )
-  (wire (pts (xy 59.69 59.69) (xy 59.69 54.61))
-    (stroke (width 0) (type default))
-  )
-  (wire (pts (xy 71.12 71.12) (xy 71.12 72.39))
+  (wire (pts (xy 59.69 57.15) (xy 59.69 52.07))
+    (stroke (width 0) (type default))
+  )
+  (wire (pts (xy 71.12 68.58) (xy 71.12 69.85))
+    (stroke (width 0) (type default))
+  )
+  (wire (pts (xy 83.82 60.96) (xy 106.68 60.96))
+    (stroke (width 0) (type default))
+  )
+  (wire (pts (xy 83.82 120.65) (xy 106.68 120.65))
+    (stroke (width 0) (type default))
+  )
+  (wire (pts (xy 46.99 129.54) (xy 46.99 97.79))
+    (stroke (width 0) (type default))
+  )
+  (wire (pts (xy 83.82 125.73) (xy 106.68 125.73))
+    (stroke (width 0) (type default))
+  )
+  (wire (pts (xy 53.34 120.65) (xy 55.88 120.65))
+    (stroke (width 0) (type default))
+  )
+  (wire (pts (xy 63.5 97.79) (xy 66.04 97.79))
+    (stroke (width 0) (type default))
+  )
+  (wire (pts (xy 60.96 93.98) (xy 60.96 97.79))
     (stroke (width 0) (type default))
   )
@@
     (stroke (width 0) (type default))
   )
-  (wire (pts (xy 83.82 120.65) (xy 106.68 120.65))
-    (stroke (width 0) (type default))
-  )
-  (wire (pts (xy 46.99 129.54) (xy 46.99 97.79))
-    (stroke (width 0) (type default))
-  )
-  (wire (pts (xy 83.82 125.73) (xy 106.68 125.73))
-    (stroke (width 0) (type default))
-  )
-  (wire (pts (xy 53.34 120.65) (xy 55.88 120.65))
-    (stroke (width 0) (type default))
-  )
-  (wire (pts (xy 63.5 97.79) (xy 66.04 97.79))
-    (stroke (width 0) (type default))
-  )
-  (wire (pts (xy 60.96 93.98) (xy 60.96 97.79))
-    (stroke (width 0) (type default))
-  )
-  (wire (pts (xy 83.82 66.04) (xy 106.68 66.04))
-    (stroke (width 0) (type default))
-  )
-  (wire (pts (xy 71.12 54.61) (xy 71.12 55.88))
+  (wire (pts (xy 71.12 52.07) (xy 71.12 53.34))
     (stroke (width 0) (type default))
   )
@@
     (stroke (width 0) (type default))
   )
-  (rectangle (start 39.37 40.64) (end 95.25 82.55)
+  (rectangle (start 39.37 38.1) (end 95.25 80.01)
     (stroke (width 0) (type default))
     (fill (type none))
@@
     (effects (font (size 1.27 1.27)) (justify left bottom))
   )
-  (text "I2C ADDR : Ox40\n(default)" (at 77.47 76.2 0)
+  (text "I2C ADDR : Ox40\n(default)" (at 77.47 73.66 0)
     (effects (font (size 1.27 1.27)) (justify left bottom))
   )
@@
     (effects (font (size 1.27 1.27)) (justify left bottom))
   )
-  (text "Humidity and Temperature Sensor" (at 44.45 44.45 0)
-    (effects (font (size 1.27 1.27)) (justify left bottom))
-  )
-  (label "I2C.SDA" (at 99.06 66.04 0) (fields_autoplaced)
+  (text "Humidity and Temperature Sensor" (at 44.45 41.91 0)
+    (effects (font (size 1.27 1.27)) (justify left bottom))
+  )
+  (label "I2C.SDA" (at 99.06 63.5 0) (fields_autoplaced)
     (effects (font (size 1.27 1.27)) (justify left bottom))
   )
@@
     (effects (font (size 1.27 1.27)) (justify left bottom))
   )
-  (label "I2C.SCL" (at 99.06 63.5 0) (fields_autoplaced)
+  (label "I2C.SCL" (at 99.06 60.96 0) (fields_autoplaced)
     (effects (font (size 1.27 1.27)) (justify left bottom))
   )
@@
     (effects (font (size 1.27 1.27)) (justify left))
   )
-  (symbol (lib_id "power:+3V3") (at 71.12 52.07 0) (unit 1)
+  (symbol (lib_id "power:+3V3") (at 71.12 49.53 0) (unit 1)
     (in_bom yes) (on_board yes) (dnp no) (fields_autoplaced)
-    (property "Reference" "#PWR04" (at 71.12 55.88 0)
-      (effects (font (size 1.27 1.27)) hide)
-    )
-    (property "Value" "+3V3" (at 71.12 48.125 0)
-      (effects (font (size 1.27 1.27)))
-    )
-    (property "Footprint" "" (at 71.12 52.07 0)
-      (effects (font (size 1.27 1.27)) hide)
-    )
-    (property "Datasheet" "" (at 71.12 52.07 0)
+    (property "Reference" "#PWR04" (at 71.12 53.34 0)
+      (effects (font (size 1.27 1.27)) hide)
+    )
+    (property "Value" "+3V3" (at 71.12 45.585 0)
+      (effects (font (size 1.27 1.27)))
+    )
+    (property "Footprint" "" (at 71.12 49.53 0)
+      (effects (font (size 1.27 1.27)) hide)
+    )
+    (property "Datasheet" "" (at 71.12 49.53 0)
       (effects (font (size 1.27 1.27)) hide)
     )
@@
     )
   )
-  (symbol (lib_id "New_Library:HTU21D") (at 73.66 63.5 0) (unit 1)
+  (symbol (lib_id "New_Library:HTU21D") (at 73.66 60.96 0) (unit 1)
     (in_bom yes) (on_board yes) (dnp no)
-    (property "Reference" "U3" (at 76.2 54.61 0)
+    (property "Reference" "U3" (at 76.2 52.07 0)
       (effects (font (size 1.27 1.27)) (justify right))
     )
-    (property "Value" "HTU21D" (at 81.28 57.15 0)
+    (property "Value" "HTU21D" (at 81.28 54.61 0)
       (effects (font (size 1.27 1.27)) (justify right))
     )
-    (property "Footprint" "" (at 71.12 86.995 0)
-      (effects (font (size 1.27 1.27)) hide)
-    )
-    (property "Datasheet" "" (at 74.93 81.28 0)
+    (property "Footprint" "" (at 71.12 84.455 0)
+      (effects (font (size 1.27 1.27)) hide)
+    )
+    (property "Datasheet" "" (at 74.93 78.74 0)
       (effects (font (size 1.27 1.27)) hide)
     )
@@
     )
   )
-  (symbol (lib_id "power:GND") (at 71.12 74.93 0) (unit 1)
+  (symbol (lib_id "power:GND") (at 71.12 72.39 0) (unit 1)
     (in_bom yes) (on_board yes) (dnp no) (fields_autoplaced)
-    (property "Reference" "#PWR06" (at 71.12 81.28 0)
-      (effects (font (size 1.27 1.27)) hide)
-    )
-    (property "Value" "GND" (at 71.12 78.875 0)
-      (effects (font (size 1.27 1.27)))
-    )
-    (property "Footprint" "" (at 71.12 74.93 0)
-      (effects (font (size 1.27 1.27)) hide)
-    )
-    (property "Datasheet" "" (at 71.12 74.93 0)
+    (property "Reference" "#PWR06" (at 71.12 78.74 0)
+      (effects (font (size 1.27 1.27)) hide)
+    )
+    (property "Value" "GND" (at 71.12 76.335 0)
+      (effects (font (size 1.27 1.27)))
+    )
+    (property "Footprint" "" (at 71.12 72.39 0)
+      (effects (font (size 1.27 1.27)) hide)
+    )
+    (property "Datasheet" "" (at 71.12 72.39 0)
       (effects (font (size 1.27 1.27)) hide)
     )
@@
     )
   )
-  (symbol (lib_id "Device:C") (at 59.69 63.5 0) (unit 1)
+  (symbol (lib_id "Device:C") (at 59.69 60.96 0) (unit 1)
     (in_bom yes) (on_board yes) (dnp no)
-    (property "Reference" "C21" (at 62.611 62.476 0)
+    (property "Reference" "C21" (at 62.611 59.936 0)
       (effects (font (size 1.27 1.27)) (justify left))
     )
-    (property "Value" "100nF" (at 62.611 64.524 0)
+    (property "Value" "100nF" (at 62.611 61.984 0)
       (effects (font (size 1.27 1.27)) (justify left))
     )
-    (property "Footprint" "Capacitor_SMD:C_0603_1608Metric" (at 60.6552 67.31 0)
-      (effects (font (size 1.27 1.27)) hide)
-    )
-    (property "Datasheet" "~" (at 59.69 63.5 0)
-      (effects (font (size 1.27 1.27)) hide)
-    )
+    (property "Footprint" "Capacitor_SMD:C_0603_1608Metric" (at 60.6552 64.77 0)
+      (effects (font (size 1.27 1.27)) hide)
+    )
+    (property "Datasheet" "~" (at 59.69 60.96 0)
+      (effects (font (size 1.27 1.27)) hide)
+    )

Commit message: udpate pcb design
Parts:
- U2: footprint (none) -> Package_DFN_QFN:Panasonic_HQFN-16-1EP_4x4mm_P0.65mm_EP2.9x2.9mm
- U3: footprint (none) -> Package_DFN_QFN:DFN-6-1EP_3x3mm_P1mm_EP1.5x2.4mm
Changed lines of the file:
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@@
       (effects (font (size 1.27 1.27)) (justify right))
     )
-    (property "Footprint" "" (at 71.12 84.455 0)
+    (property "Footprint" "Package_DFN_QFN:DFN-6-1EP_3x3mm_P1mm_EP1.5x2.4mm" (at 71.12 84.455 0)
       (effects (font (size 1.27 1.27)) hide)
     )
@@
       (effects (font (size 1.27 1.27)))
     )
-    (property "Footprint" "" (at 60.325 108.585 0)
+    (property "Footprint" "Package_DFN_QFN:Panasonic_HQFN-16-1EP_4x4mm_P0.65mm_EP2.9x2.9mm" (at 60.325 108.585 0)
       (effects (font (size 1.27 1.27)) hide)
     )
