File: hardware/OpenWeatherStation_MainBoard/OpenWeatherStation_MainBoard.kicad_pcb (KiCad board)
At the start: 2 copper layers, 50.8 x 101.6 mm, 91 parts, among them J4 Conn_02x07_Odd_Even, U1 STM32F107VCTx, U10 TL431DBV, U7 USBLC6-4SC6, U8 LAN8742A, U9 TCMT1107, Y1 Crystal

Commit message: udpate pcb design
Parts:
- added C1: 100nF, Capacitor_SMD:C_0603_1608Metric, F.Cu at (80.1, 91.5)
- added C2: 100nF, Capacitor_SMD:C_0603_1608Metric, F.Cu at (80.1, 94.0)
- added C3: 100nF, Capacitor_SMD:C_0603_1608Metric, F.Cu at (80.1, 96.6)
- added C4: 100nF, Capacitor_SMD:C_0603_1608Metric, F.Cu at (80.1, 99.1)
- added C5: 100nF, Capacitor_SMD:C_0603_1608Metric, F.Cu at (80.1, 101.6)
- added C9: 100nF, Capacitor_SMD:C_0603_1608Metric, F.Cu at (80.1, 104.1)
- added D10: SMAJ58A, Diode_SMD:D_SMA, F.Cu at (143.4, 175.0)
- added D12: D_Schottky, Diode_SMD:D_1206_3216Metric, F.Cu at (123.6, 169.5)
- added D4: D_Schottky, Diode_SMD:D_PowerDI-5, F.Cu at (135.0, 175.5)
- added D9: D_Schottky, Diode_SMD:D_1206_3216Metric, F.Cu at (123.6, 166.1)
- added FB1: FerriteBead, Capacitor_SMD:C_0603_1608Metric, F.Cu at (86.1, 104.0)
- added FB2: FerriteBead, Capacitor_SMD:C_0603_1608Metric, F.Cu at (80.1, 106.6)
- added J2: Conn_01x05_Pin, Connector_JST:JST_XH_B5B-XH-A_1x05_P2.50mm_Vertical, F.Cu at (99.0, 84.3)
- added J3: RJ45_LED_Shielded, Connector_RJ:RJ45_Amphenol_RJHSE538X, F.Cu at (90.9, 170.2)
- added Q1: Q_NMOS_GDS, Package_TO_SOT_SMD:TO-252-2, F.Cu at (137.6, 168.7)
- added R3: 158R, Resistor_SMD:R_0603_1608Metric, F.Cu at (122.8, 179.1)
- added U2: FXPS7115D4, Package_DFN_QFN:Panasonic_HQFN-16-1EP_4x4mm_P0.65mm_EP2.9x2.9mm, F.Cu at (87.1, 90.8)
- added U3: HTU21D, Package_DFN_QFN:DFN-6-1EP_3x3mm_P1mm_EP1.5x2.4mm, F.Cu at (86.7, 98.5)
- added U4: ~, Transformer_SMD:Transformer_Ethernet_Wuerth_749013011A, F.Cu at (63.5, 162.6)
- added U5: PM8800A, Package_SO:HTSSOP-16-1EP_4.4x5mm_P0.65mm_EP3x3mm, F.Cu at (125.2, 174.5)
- added U6: POE13P-33L, Library:SM13117EL, F.Cu at (134.6, 152.4)
- moved C39 9.72 mm to (80.9, 154.9)
Connections:
- C35 pad 2: Net-(D7-K) -> Net-(D4-K)
- C36 pad 2: Net-(D7-K) -> Net-(D4-K)
- C37 pad 2: Net-(D7-K) -> Net-(D4-K)
- L2 pad 1: Net-(D7-K) -> Net-(D4-K)
- U1 pad 19: unconnected-(U1-VSSA-Pad19) -> GND
- U1 pad 21: unconnected-(U1-VREF+-Pad21) -> +3.3VA
- U1 pad 22: unconnected-(U1-VDDA-Pad22) -> +3.3VA
- U1 pad 6: unconnected-(U1-VBAT-Pad6) -> +3V3

Commit message: update pcb
Parts:
- removed R13: 0.33R, Resistor_SMD:R_0603_1608Metric
- C1, C16, C17, C2, C25, C26, C27, C28, C29, C3, C30, C31, C32, C4, C5, C9, D1, D2, Q1, R15, R20, R21, R22, R23, R25, R31, R32, R33, R34, R35, R36, R37, R9: moved to B.Cu
- C36, C37, C38: footprint Capacitor_SMD:CP_Elec_5x3 -> Capacitor_SMD:C_0603_1608Metric
- R11: footprint Resistor_SMD:R_0603_1608Metric -> Resistor_SMD:R_1206_3216Metric
- moved D4 63.6 mm to (91.8, 128.8), turned to 180 degrees
- moved U4 57.5 mm to (117.5, 142.8), turned to -90 degrees
- moved D10 56.4 mm to (90.0, 157.0), turned to 90 degrees
- moved C6 53.2 mm to (100.0, 185.1), turned to -90 degrees
- moved JP1 52.4 mm to (94.7, 115.2), turned to 90 degrees
- moved C7 50.4 mm to (96.8, 185.1), turned to -90 degrees
- moved C11 50.2 mm to (80.0, 184.0), turned to -90 degrees
- moved Q1 50.0 mm to (89.0, 157.0), turned to 90 degrees
- moved U6 49.8 mm to (85.8, 142.7)
- moved D1 47.7 mm to (96.0, 180.0)
- moved C10 45.2 mm to (93.7, 185.0), turned to -90 degrees
- moved D9 44.9 mm to (80.0, 155.9), turned to 90 degrees
- moved U5 42.5 mm to (83.0, 169.2), turned to 180 degrees
- moved R9 42.0 mm to (82.8, 172.0)
- moved L2 38.3 mm to (85.7, 128.8), turned to -90 degrees
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Connections:
- U5 pad 1: (no net) -> Net-(U5-RT)
- U5 pad 10: (no net) -> Net-(U5-GD)
- U5 pad 11: (no net) -> Net-(D9-K)
- U5 pad 12: (no net) -> Net-(D5-K)
- U5 pad 13: (no net) -> Net-(U5-CS)
- U5 pad 14: (no net) -> Net-(U5-COMP)
- U5 pad 15: (no net) -> GNDA
- U5 pad 16: (no net) -> GNDA
- U5 pad 2: (no net) -> Net-(U5-SS)
- U5 pad 3: (no net) -> unconnected-(U5-AUXII-Pad3)
- U5 pad 4: (no net) -> /PoE/VIN
- U5 pad 5: (no net) -> Net-(U5-RCLASS)
- U5 pad 6: (no net) -> unconnected-(U5-AUXI_IRL-Pad6)
- U5 pad 7: (no net) -> Net-(U5-DCCL)
- U5 pad 8: (no net) -> /PoE/VSS
- U5 pad 9: (no net) -> GNDPWR
- U6 pad 10: (no net) -> Net-(D8-K)
- U6 pad 2: GND -> GNDA
- U6 pad 5: Net-(D4-A) -> (no net)
- U6 pad 6: Net-(D4-A) -> (no net)
- U6 pad 7: Net-(D8-K) -> Net-(D4-A)
- U6 pad 8: Net-(D8-K) -> Net-(D4-A)
- U6 pad 9: (no net) -> Net-(D8-K)
Routing:
- added copper zone on B.Cu, net GND
- added copper zone on F.Cu, net GND
Other:
- board size 50.8 x 101.6 mm -> 50 x 100 mm
