File: hardware/OpenWeatherStation_MainBoard/untitled.kicad_sch (KiCad schematic)
At the start: 50 parts, among them Q1 Q_NMOS_GDS, U5 PM8800A, U6 POE13P-33L

Commit message: poe wip
Parts:
- removed C1, C15, C2, C3, C4, C9: 1nF, symbol Device:C
- removed C5: 2.2nF, symbol Device:C
- removed R10: 52R, symbol Device:R
- removed R3, R4, R5, R6: 75, symbol Device:R
- added C34, C40, C41: 1uF, symbol Device:C
- added C35: 560pF, symbol Device:C
- added C36, C37, C38: 22uF, symbol Device:C
- added C39: 330uF, symbol Device:C_Polarized
- added C42: 22nF, symbol Device:C
- added D11, D7: D, symbol Device:D
- added D12: D_Schottky, symbol Device:D_Schottky
- added D8: LED, symbol Device:LED
- added JP1: SolderJumper_2_Open, symbol Jumper:SolderJumper_2_Open
- added L2: L, symbol Device:L
- added R29: 10k, symbol Device:R
- added R30: 4R7, Resistor_SMD:R_1206_3216Metric, symbol Device:R
- added R39: 21k, symbol Device:R
- added R40: 12.4k, symbol Device:R
- added R41: 10R, symbol Device:R
- added R42: 390R, symbol Device:R
- added R44: 3k3, symbol Device:R
- added U10: TL431DBV, Package_TO_SOT_SMD:SOT-23-5, symbol Reference_Voltage:TL431DBV
- added U9: TCMT1107, Package_SO:SOP-4_4.4x2.6mm_P1.27mm, symbol Isolator:TCMT1107
- C8: value 1nF -> 2n2
- R15: value 510R -> 100
- R8: value 10R -> 1k
Connections:
- net GND: now also U6.1, C40.1, R40.2, U10.5 (A); no longer C14.2, C17.2, C20.2, R11.1, R14.1, U5. (nPGD), U6.4
- net GNDA: now also C16.2, R9.1, U5. (nPGD), C34.2, U9.3
- net GNDPWR: now also C11.2, C12.2, C13.2, C14.2, C17.2, C20.2, C8.1, R11.1, R14.1, U5. (nPGD)
- net VSS: no longer C11.2, C12.2, C13.2
- net at C12.1, C13.1, L1.2: now also U6.3, D12.2 (A); no longer R8.1, U6.2
- net at R8.2: now also D8.2 (A); no longer U5. (nPGD)
- net at Q1.2 (D): now also U6.4, D11.2 (A); no longer U6.1
- net at R17.2: now also U6.2; no longer U6.3
- net at U6.5, U6.6: now also D7.2 (A), R30.2
- net at U6.7, U6.8: now also C36.1, C37.1, C38.1, C39.2, D8.1 (K)
- net POE_F renamed VIN
- net VIN: now also U5. (nPGD); no longer C8.1
- new net: D11.1 (K), D12.1 (K)
- new net: R9.2, U5. (nPGD)
- new net: C41.1, R39.2, R40.1, R44.2, U10.4 (REF)
- new net: C40.2, R41.1, U9.1
- new net: C38.2, C39.1, JP1.1 (A), L2.2, R39.1, R41.2, R8.1
- new net: C34.1, R29.1
- new net: R29.2, U5. (nPGD), U9.4
- new net: R42.1, U9.2
- new net: C35.1, R30.1
- new net: C35.2, C36.2, C37.2, D7.1 (K), L2.1
- new net: C42.1, R44.1
- new net: C41.2, C42.2, R42.2, U10.3 (K)
- new net: C16.1, U5. (nPGD)
- new net +3.3V: JP1.2 (B)
- no-connect marks 0 -> 1
Other:
- moved on the sheet: C10, C11, C12, C13, C14, C16, C17, C18, C19, C20, C6, C7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

Commit message: electrical design wip
Parts:
- C10, C12, C13, C16, C19: value 0.1uF -> 100nF; footprint (none) -> Capacitor_SMD:C_0603_1608Metric
- C11, C36, C37, C38, C39: footprint (none) -> Capacitor_SMD:CP_Elec_5x3
- C14, C17, C18, C20, C34, C35, C40, C41, C42, C6, C7: footprint (none) -> Capacitor_SMD:C_0603_1608Metric
- C8: value 2n2 -> 2.2nF; footprint (none) -> Capacitor_SMD:C_0603_1608Metric
- D5, D8: footprint (none) -> LED_THT:LED_D3.0mm
- JP1: footprint (none) -> Jumper:SolderJumper-2_P1.3mm_Open_RoundedPad1.0x1.5mm
- L1, L2: footprint (none) -> Inductor_SMD:L_1206_3216Metric
- R11, R12, R13, R14, R16, R17, R29, R39, R41, R42, R44, R7, R8, R9: footprint (none) -> Resistor_SMD:R_0603_1608Metric
- R15: value 100 -> 100R; footprint (none) -> Resistor_SMD:R_0603_1608Metric
- R30: footprint Resistor_SMD:R_1206_3216Metric -> Resistor_SMD:R_0603_1608Metric
- R40: value 12.4k -> 12k4; footprint (none) -> Resistor_SMD:R_0603_1608Metric
Other:
- company: (none) -> Vital Septfonds
- title: (none) -> Open Wheather Station

Commit message: update elec
Parts:
- removed D11, D4, D6, D7: D, symbol Device:D
- removed R13: 0.33R, Resistor_SMD:R_0603_1608Metric, symbol Device:R
- added D10: SMAJ58A, Diode_SMD:D_SMA, symbol Diode:SMAJ58A
- added D4, D9: D_Schottky, symbol Device:D_Schottky
Connections:
- net GND: now also U6.2; no longer U6.1
- net at D12.1 (K): now also D10.1 (A1)
- net at Q1.2 (D), U6.4: now also D10.2 (A2)
- net at C19.1, C20.1, R16.2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: now also D9.1 (K)
- net at C35.2, C36.2, C37.2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: now also D4.1 (K)
- net at R17.2: now also U6.1; no longer U6.2
- net at R30.2, U6.5, U6.6: now also D4.2 (A)
- net at R17.1: now also D9.2 (A)
Other:
- note added: "Primary"
- note added: "Secondary"
- moved on the sheet: C10, C11, C12, C13, C14, C16, C17, C18, C19, C20, C34, C35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

Commit message: udpate pcb design
Parts:
- added R3: 158R, Resistor_SMD:R_0603_1608Metric, symbol Device:R
- D12, D9: footprint (none) -> Diode_SMD:D_1206_3216Metric
- D4: footprint (none) -> Diode_SMD:D_PowerDI-5
- Q1: footprint (none) -> Package_TO_SOT_SMD:TO-252-2
- U4: footprint (none) -> Transformer_SMD:Transformer_Ethernet_Wuerth_749013011A
- U5: footprint (none) -> Package_SO:HTSSOP-16-1EP_4.4x5mm_P0.65mm_EP3x3mm
- U6: footprint (none) -> Library:SM13117EL
Connections:
- net VSS: now also R3.2
- new net: R3.1, U5. (nPGD)
- no-connect marks 1 -> 2
Other:
- moved on the sheet: R7
Changed lines of the file:
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@@
   (junction (at 198.12 198.12) (diameter 0) (color 0 0 0 0)
   )
+  (junction (at 118.11 209.55) (diameter 0) (color 0 0 0 0)
+  )
   (junction (at 307.34 134.62) (diameter 0) (color 0 0 0 0)
   )
@@
   (junction (at 148.59 130.81) (diameter 0) (color 0 0 0 0)
   )
-  (junction (at 111.76 209.55) (diameter 0) (color 0 0 0 0)
-  )
   (junction (at 170.18 144.78) (diameter 0) (color 0 0 0 0)
   )
@@
   (junction (at 321.31 134.62) (diameter 0) (color 0 0 0 0)
   )
+  (junction (at 109.22 209.55) (diameter 0) (color 0 0 0 0)
+  )
   (junction (at 133.35 66.04) (diameter 0) (color 0 0 0 0)
   )
@@
   (junction (at 198.12 209.55) (diameter 0) (color 0 0 0 0)
   )
-  (no_connect (at 132.08 187.96))
+  (no_connect (at 132.08 180.34))
+  (no_connect (at 132.08 175.26))
   (bus_entry (at 273.05 44.45) (size 2.54 2.54)
     (stroke (width 0) (type default))
@@
     (stroke (width 0) (type default))
   )
+  (wire (pts (xy 132.08 187.96) (xy 118.11 187.96))
+    (stroke (width 0) (type default))
+  )
   (wire (pts (xy 307.34 134.62) (xy 302.26 134.62))
     (stroke (width 0) (type default))
@@
     (stroke (width 0) (type default))
   )
+  (wire (pts (xy 118.11 187.96) (xy 118.11 195.58))
+    (stroke (width 0) (type default))
+  )
   (bus (pts (xy 45.72 73.66) (xy 45.72 71.12))
     (stroke (width 0) (type default))
@@
     (stroke (width 0) (type default))
   )
-  (wire (pts (xy 132.08 185.42) (xy 111.76 185.42))
+  (wire (pts (xy 132.08 185.42) (xy 109.22 185.42))
     (stroke (width 0) (type default))
   )
@@
     (stroke (width 0) (type default))
   )
-  (wire (pts (xy 100.33 209.55) (xy 111.76 209.55))
-    (stroke (width 0) (type default))
-  )
   (wire (pts (xy 69.85 66.04) (xy 71.12 66.04))
     (stroke (width 0) (type default))
@@
     (stroke (width 0) (type default))
   )
-  (wire (pts (xy 111.76 185.42) (xy 111.76 195.58))
+  (wire (pts (xy 109.22 185.42) (xy 109.22 195.58))
     (stroke (width 0) (type default))
   )
@@
     (stroke (width 0) (type default))
   )
-  (wire (pts (xy 111.76 209.55) (xy 127 209.55))
-    (stroke (width 0) (type default))
-  )
   (wire (pts (xy 198.12 175.26) (xy 198.12 198.12))
     (stroke (width 0) (type default))
@@
     (stroke (width 0) (type default))
   )
+  (wire (pts (xy 92.71 209.55) (xy 109.22 209.55))
+    (stroke (width 0) (type default))
+  )
   (wire (pts (xy 53.34 148.59) (xy 53.34 160.02))
     (stroke (width 0) (type default))
@@
     (stroke (width 0) (type default))
   )
+  (wire (pts (xy 109.22 209.55) (xy 118.11 209.55))
+    (stroke (width 0) (type default))
+  )
   (wire (pts (xy 81.28 71.12) (xy 81.28 66.04))
     (stroke (width 0) (type default))
@@
     (stroke (width 0) (type default))
   )
+  (wire (pts (xy 118.11 209.55) (xy 127 209.55))
+    (stroke (width 0) (type default))
+  )
   (wire (pts (xy 187.96 170.18) (xy 187.96 182.88))
     (stroke (width 0) (type default))
@@
     (stroke (width 0) (type default))
   )
-  (wire (pts (xy 111.76 203.2) (xy 111.76 209.55))
+  (wire (pts (xy 109.22 203.2) (xy 109.22 209.55))
     (stroke (width 0) (type default))
   )
@@
   )
   (wire (pts (xy 323.85 199.39) (xy 327.66 199.39))
+    (stroke (width 0) (type default))
+  )
+  (wire (pts (xy 118.11 203.2) (xy 118.11 209.55))
     (stroke (width 0) (type default))
   )
@@
     (effects (font (size 1.27 1.27)) (justify right bottom))
   )
-  (label "VSS" (at 100.33 209.55 0) (fields_autoplaced)
+  (label "VSS" (at 92.71 209.55 0) (fields_autoplaced)
     (effects (font (size 1.27 1.27)) (justify left bottom))
   )
@@
       (effects (font (size 1.27 1.27)) (justify right))
     )
-    (property "Footprint" "" (at 180.34 144.78 0)
+    (property "Footprint" "Diode_SMD:D_1206_3216Metric" (at 180.34 144.78 0)
       (effects (font (size 1.27 1.27)) hide)
     )
@@
       (effects (font (size 1.27 1.27)) (justify left))
     )
-    (property "Footprint" "" (at 200.66 167.64 0)
+    (property "Footprint" "Package_TO_SOT_SMD:TO-252-2" (at 200.66 167.64 0)
       (effects (font (size 1.27 1.27)) hide)
     )
@@
       (effects (font (size 1.27 1.27)))
     )
-    (property "Footprint" "" (at 240.03 137.16 0)
+    (property "Footprint" "Library:SM13117EL" (at 240.03 137.16 0)
       (effects (font (size 1.27 1.27)) hide)
     )
@@
       (effects (font (size 1.27 1.27)) (justify right))
     )
-    (property "Footprint" "" (at 168.91 137.16 0)
+    (property "Footprint" "Diode_SMD:D_1206_3216Metric" (at 168.91 137.16 0)
       (effects (font (size 1.27 1.27)) hide)
     )
@@
       (effects (font (size 1.27 1.27)))
     )
-    (property "Footprint" "" (at 236.22 46.355 0)
+    (property "Footprint" "Transformer_SMD:Transformer_Ethernet_Wuerth_749013011A" (at 236.22 46.355 0)
       (effects (font (size 1.27 1.27)) hide)
     )
@@
       (effects (font (size 1.27 1.27)))
     )
-    (property "Footprint" "" (at 142.24 177.8 0)
+    (property "Footprint" "Package_SO:HTSSOP-16-1EP_4.4x5mm_P0.65mm_EP3x3mm" (at 142.24 177.8 0)
       (effects (font (size 1.27 1.27)) hide)
     )
@@
       (effects (font (size 1.27 1.27)) (justify right))
     )
-    (property "Footprint" "" (at 261.62 134.62 0)
+    (property "Footprint" "Diode_SMD:D_PowerDI-5" (at 261.62 134.62 0)
       (effects (font (size 1.27 1.27)) hide)
     )
@@
     )
   )
-  (symbol (lib_id "Device:R") (at 111.76 199.39 0) (unit 1)
-    (in_bom yes) (on_board yes) (dnp no) (fields_autoplaced)
-    (property "Reference" "R7" (at 114.3 198.12 0)
-      (effects (font (size 1.27 1.27)) (justify left))
-    )
-    (property "Value" "22k" (at 114.3 200.66 0)
-      (effects (font (size 1.27 1.27)) (justify left))
-    )
-    (property "Footprint" "Resistor_SMD:R_0603_1608Metric" (at 109.982 199.39 90)
-      (effects (font (size 1.27 1.27)) hide)
-    )
-    (property "Datasheet" "~" (at 111.76 199.39 0)
+  (symbol (lib_id "Device:R") (at 109.22 199.39 0) (unit 1)
+    (in_bom yes) (on_board yes) (dnp no) (fields_autoplaced)
+    (property "Reference" "R7" (at 111.76 198.12 0)
+      (effects (font (size 1.27 1.27)) (justify left))
+    )
+    (property "Value" "22k" (at 111.76 200.66 0)
+      (effects (font (size 1.27 1.27)) (justify left))
+    )
+    (property "Footprint" "Resistor_SMD:R_0603_1608Metric" (at 107.442 199.39 90)
+      (effects (font (size 1.27 1.27)) hide)
+    )
+    (property "Datasheet" "~" (at 109.22 199.39 0)
       (effects (font (size 1.27 1.27)) hide)
     )
@@
         )
       )
+    )
+  )
+  (symbol (lib_id "Device:R") (at 118.11 199.39 0) (unit 1)
+    (in_bom yes) (on_board yes) (dnp no) (fields_autoplaced)
+    (property "Reference" "R3" (at 120.65 198.12 0)
+      (effects (font (size 1.27 1.27)) (justify left))
+    )
+    (property "Value" "158R" (at 120.65 200.66 0)
+      (effects (font (size 1.27 1.27)) (justify left))
+    )
+    (property "Footprint" "Resistor_SMD:R_0603_1608Metric" (at 116.332 199.39 90)
+      (effects (font (size 1.27 1.27)) hide)
+    )
+    (property "Datasheet" "~" (at 118.11 199.39 0)
+      (effects (font (size 1.27 1.27)) hide)
+    )
+    (pin "1")
+    (pin "2")
+    (instances
+      (project "OpenWeatherStation_MainBoard"
+        (path "/698c4dde-56a2-4dd1-89d2-180a09a5dfe9/7c03bbc1-3816-4af6-9da6-b1bc735a9c60"
+          (reference "R3") (unit 1)
+        )
+      )

Commit message: update pcb
Parts:
- C36, C37, C38: footprint Capacitor_SMD:CP_Elec_5x3 -> Capacitor_SMD:C_0603_1608Metric
- R11: footprint Resistor_SMD:R_0603_1608Metric -> Resistor_SMD:R_1206_3216Metric
Connections:
- net GND: no longer U6.2
- net GNDA: now also U5.15 (VFB), U5.16 (AGND), U6.2; no longer U5. (nPGD)
- net GNDPWR: now also U5.9 (GND); no longer U5. (nPGD)
- net VIN: now also U5.4 (VIN); no longer U5. (nPGD)
- net VSS: now also U5.8 (VSS); no longer U5. (nPGD)
- net at R9.2: now also U5.1 (RT); no longer U5. (nPGD)
- net at C19.1, C20.1, D9.1 (K)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: now also U5.11 (VCC); no longer U5. (nPGD)
- net at R29.2, U9.4: now also U5.14 (COMP); no longer U5. (nPGD)
- net at C36.1, C37.1, C38.1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: now also U6.10, U6.9; no longer U6.7, U6.8
- net at C17.1, R15.2: now also U5.13 (CS); no longer U5. (nPGD)
- net at D4.2 (A), R30.2: now also U6.7, U6.8; no longer U6.5, U6.6
- net at C16.1: now also U5.2 (SS); no longer U5. (nPGD)
- net at C18.1, D5.1 (K): now also U5.12 (nPGD); no longer U5. (nPGD)
- net at R7.1: now also U5.7 (DCCL); no longer U5. (nPGD)
- net at R3.1: now also U5.5 (RCLASS); no longer U5. (nPGD)
- net at R12.2: now also U5.10 (GD); no longer U5. (nPGD)
Changed lines of the file:
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@@
     (pin "3")
     (pin "4")
-    (pin "5")
-    (pin "6")
+    (pin "10")
+    (pin "9")
     (pin "7")
     (pin "8")
@@
       (effects (font (size 1.27 1.27)) (justify right))
     )
-    (property "Footprint" "Capacitor_SMD:CP_Elec_5x3" (at 277.1648 138.43 0)
+    (property "Footprint" "Capacitor_SMD:C_0603_1608Metric" (at 277.1648 138.43 0)
       (effects (font (size 1.27 1.27)) hide)
     )
@@
       (effects (font (size 1.27 1.27)) (justify right))
     )
-    (property "Footprint" "Capacitor_SMD:CP_Elec_5x3" (at 306.3748 138.43 0)
+    (property "Footprint" "Capacitor_SMD:C_0603_1608Metric" (at 306.3748 138.43 0)
       (effects (font (size 1.27 1.27)) hide)
     )
@@
     )
   )
-  (symbol (lib_id "power:GND") (at 231.14 156.21 0) (unit 1)
-    (in_bom yes) (on_board yes) (dnp no) (fields_autoplaced)
-    (property "Reference" "#PWR014" (at 231.14 162.56 0)
-      (effects (font (size 1.27 1.27)) hide)
-    )
-    (property "Value" "GND" (at 231.14 160.155 0)
-      (effects (font (size 1.27 1.27)))
-    )
-    (property "Footprint" "" (at 231.14 156.21 0)
-      (effects (font (size 1.27 1.27)) hide)
-    )
-    (property "Datasheet" "" (at 231.14 156.21 0)
-      (effects (font (size 1.27 1.27)) hide)
-    )
-    (pin "1")
-    (instances
-      (project "OpenWeatherStation_MainBoard"
-        (path "/698c4dde-56a2-4dd1-89d2-180a09a5dfe9/7c03bbc1-3816-4af6-9da6-b1bc735a9c60"
-          (reference "#PWR014") (unit 1)
-        )
-      )
-    )
-  )
   (symbol (lib_id "Device:C") (at 175.26 204.47 0) (unit 1)
     (in_bom yes) (on_board yes) (dnp no) (fields_autoplaced)
@@
       (effects (font (size 1.27 1.27)) (justify right))
     )
-    (property "Footprint" "Resistor_SMD:R_0603_1608Metric" (at 199.898 203.2 90)
+    (property "Footprint" "Resistor_SMD:R_1206_3216Metric" (at 199.898 203.2 90)
       (effects (font (size 1.27 1.27)) hide)
     )
@@
       (effects (font (size 1.27 1.27)) hide)
     )
-    (pin "")
-    (pin "")
-    (pin "")
-    (pin "")
-    (pin "")
-    (pin "")
-    (pin "")
-    (pin "")
-    (pin "")
-    (pin "")
-    (pin "")
-    (pin "")
-    (pin "")
-    (pin "")
-    (pin "")
-    (pin "")
+    (pin "13")
+    (pin "5")
+    (pin "10")
+    (pin "15")
+    (pin "16")
+    (pin "4")
+    (pin "11")
+    (pin "8")
+    (pin "9")
+    (pin "3")
+    (pin "6")
+    (pin "1")
+    (pin "12")
+    (pin "7")
+    (pin "14")
+    (pin "2")
     (instances
       (project "OpenWeatherStation_MainBoard"
@@
     )
   )
+  (symbol (lib_id "power:GNDA") (at 231.14 156.21 0) (unit 1)
+    (in_bom yes) (on_board yes) (dnp no) (fields_autoplaced)
+    (property "Reference" "#PWR014" (at 231.14 162.56 0)
+      (effects (font (size 1.27 1.27)) hide)
+    )
+    (property "Value" "GNDA" (at 231.14 160.155 0)
+      (effects (font (size 1.27 1.27)))
+    )
+    (property "Footprint" "" (at 231.14 156.21 0)
+      (effects (font (size 1.27 1.27)) hide)
+    )
+    (property "Datasheet" "" (at 231.14 156.21 0)
+      (effects (font (size 1.27 1.27)) hide)
+    )
+    (pin "1")
+    (instances
+      (project "OpenWeatherStation_MainBoard"
+        (path "/698c4dde-56a2-4dd1-89d2-180a09a5dfe9/7c03bbc1-3816-4af6-9da6-b1bc735a9c60"
+          (reference "#PWR014") (unit 1)
+        )
+      )
+    )
+  )
   (symbol (lib_id "Reference_Voltage:TL431DBV") (at 323.85 204.47 270) (mirror x) (unit 1)
     (in_bom yes) (on_board yes) (dnp no)
@@
       (effects (font (size 1.27 1.27)) (justify right))
     )
-    (property "Footprint" "Capacitor_SMD:CP_Elec_5x3" (at 288.5948 138.43 0)
-      (effects (font (size 1.27 1.27)) hide)
-    )
+    (property "Footprint" "Capacitor_SMD:C_0603_1608Metric" (at 288.5948 138.43 0)
+      (effects (font (size 1.27 1.27)) hide)
+    )
